Commit message: Add configurable multi-robot simulation with ROS bridges and RViz

File: src/edgeai_robot_description/urdf/edgeai_robot_real.urdf.xacro (robot description, xacro)
@@ -2,4 +2,15 @@
 <robot xmlns:xacro="http://www.ros.org/wiki/xacro"
        name="edgeai_robot_real">
+  <!-- Multi-robot configuration -->
+  <xacro:arg name="robot_ns" default=""/>
+  <xacro:property
+    name="robot_ns"
+    value="$(arg robot_ns)"/>
+  <xacro:property
+    name="frame_prefix"
+    value="${robot_ns + '/' if robot_ns else ''}"/>
+  <xacro:property
+    name="topic_prefix"
+    value="${'/' + robot_ns if robot_ns else ''}"/>
   <!-- Parameters -->
   <!-- Lower folded-aluminum chassis -->
@@ -457,6 +468,6 @@
     <always_on>true</always_on>
     <update_rate>30</update_rate>
-    <topic>camera</topic>
-    <optical_frame_id>camera_optical_frame</optical_frame_id>
+    <topic>${topic_prefix + "/camera" if robot_ns else "camera"}</topic>
+    <optical_frame_id>${frame_prefix}camera_optical_frame</optical_frame_id>
     <camera>
       <horizontal_fov>1.047</horizontal_fov>
@@ -510,7 +521,7 @@
       <pose>0 0 0 0 0 0</pose>
       <!-- Gazebo Transport topic -->
-      <topic>/scan</topic>
+      <topic>${topic_prefix}/scan</topic>
       <!-- Frame carried in the LiDAR message -->
-      <gz_frame_id>lidar_link</gz_frame_id>
+      <gz_frame_id>${frame_prefix}lidar_link</gz_frame_id>
       <update_rate>10</update_rate>
       <lidar>
@@ -545,10 +556,10 @@
       <wheel_radius>${wheel_radius}</wheel_radius>
       <!-- Gazebo command / odometry topics -->
-      <topic>/cmd_vel</topic>
-      <odom_topic>/odom</odom_topic>
-      <tf_topic>/tf</tf_topic>
+      <topic>${topic_prefix}/cmd_vel</topic>
+      <odom_topic>${topic_prefix}/odom</odom_topic>
+      <tf_topic>${topic_prefix}/tf</tf_topic>
       <!-- Odometry frame -->
-      <frame_id>odom</frame_id>
-      <child_frame_id>base_footprint</child_frame_id>
+      <frame_id>${frame_prefix}odom</frame_id>
+      <child_frame_id>${frame_prefix}base_footprint</child_frame_id>
       <!-- Odometry publishing -->
       <odom_publish_frequency>50</odom_publish_frequency>
@@ -559,5 +570,5 @@
     filename="gz-sim-joint-state-publisher-system"
     name="gz::sim::systems::JointStatePublisher">
-    <topic>joint_states</topic>
+    <topic>${topic_prefix + "/joint_states" if robot_ns else "joint_states"}</topic>
   </plugin>
 </gazebo>

Commit message: support multiple slam at the same time

File: src/edgeai_robot_description/urdf/edgeai_robot_real.urdf.xacro (robot description, xacro)
@@ -2,15 +2,4 @@
 <robot xmlns:xacro="http://www.ros.org/wiki/xacro"
        name="edgeai_robot_real">
-  <!-- Multi-robot configuration -->
-  <xacro:arg name="robot_ns" default=""/>
-  <xacro:property
-    name="robot_ns"
-    value="$(arg robot_ns)"/>
-  <xacro:property
-    name="frame_prefix"
-    value="${robot_ns + '/' if robot_ns else ''}"/>
-  <xacro:property
-    name="topic_prefix"
-    value="${'/' + robot_ns if robot_ns else ''}"/>
   <!-- Parameters -->
   <!-- Lower folded-aluminum chassis -->
@@ -468,6 +457,6 @@
     <always_on>true</always_on>
     <update_rate>30</update_rate>
-    <topic>${topic_prefix + "/camera" if robot_ns else "camera"}</topic>
-    <optical_frame_id>${frame_prefix}camera_optical_frame</optical_frame_id>
+    <topic>camera</topic>
+    <optical_frame_id>camera_optical_frame</optical_frame_id>
     <camera>
       <horizontal_fov>1.047</horizontal_fov>
@@ -521,7 +510,7 @@
       <pose>0 0 0 0 0 0</pose>
       <!-- Gazebo Transport topic -->
-      <topic>${topic_prefix}/scan</topic>
+      <topic>/scan</topic>
       <!-- Frame carried in the LiDAR message -->
-      <gz_frame_id>${frame_prefix}lidar_link</gz_frame_id>
+      <gz_frame_id>lidar_link</gz_frame_id>
       <update_rate>10</update_rate>
       <lidar>
@@ -556,10 +545,10 @@
       <wheel_radius>${wheel_radius}</wheel_radius>
       <!-- Gazebo command / odometry topics -->
-      <topic>${topic_prefix}/cmd_vel</topic>
-      <odom_topic>${topic_prefix}/odom</odom_topic>
-      <tf_topic>${topic_prefix}/tf</tf_topic>
+      <topic>/cmd_vel</topic>
+      <odom_topic>/odom</odom_topic>
+      <tf_topic>/tf</tf_topic>
       <!-- Odometry frame -->
-      <frame_id>${frame_prefix}odom</frame_id>
-      <child_frame_id>${frame_prefix}base_footprint</child_frame_id>
+      <frame_id>odom</frame_id>
+      <child_frame_id>base_footprint</child_frame_id>
       <!-- Odometry publishing -->
       <odom_publish_frequency>50</odom_publish_frequency>
@@ -570,5 +559,5 @@
     filename="gz-sim-joint-state-publisher-system"
     name="gz::sim::systems::JointStatePublisher">
-    <topic>${topic_prefix + "/joint_states" if robot_ns else "joint_states"}</topic>
+    <topic>joint_states</topic>
   </plugin>
 </gazebo>
